File: hardware/hardware.kicad_pcb (KiCad board)
At the start: 2 copper layers, 36.8 x 67.3 mm, 53 parts, among them J1 SWD, J2 serial, J3 analog, J4 digital_0, J5 digital_1, J6 digital_2, J7 digital_3, J8 power_0, J9 power_1, SW1 reset_btn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

Commit message: ordering first prototype
Parts:
- moved C12 73.6 mm to (128.7, 110.1)
- moved R5 71.2 mm to (142.0, 94.4)
- moved R6 71.2 mm to (140.5, 94.4)
- moved R7 71.2 mm to (138.9, 94.4)
- moved C7 71.2 mm to (137.4, 94.4)
- moved J1 71.0 mm to (139.5, 80.0)
- moved R8 71.0 mm to (137.2, 83.6)
- moved U1 71.0 mm to (139.5, 108.9)
- moved C10 71.0 mm to (131.4, 87.4)
- moved C13 71.0 mm to (145.1, 114.3)
- moved C16 71.0 mm to (143.5, 114.3)
- moved C18 71.0 mm to (139.5, 125.2)
- moved C3 71.0 mm to (151.5, 86.0)
- moved C4 71.0 mm to (149.6, 85.9)
- moved C5 71.0 mm to (136.3, 88.6)
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Connections:
- J4 pad 1: PA12 -> PA10
- J4 pad 2: PA11 -> PA9
- J4 pad 3: PA10 -> PA8
- J4 pad 4: PA9 -> PB15
- J4 pad 5: PA8 -> PB14
- J5 pad 1: PB5 -> PB4
- J5 pad 2: PB4 -> PB3
- J5 pad 3: PB3 -> PA15
- J5 pad 4: PA15 -> PA12
- J5 pad 5: PB2 -> PA11
- J6 pad 1: PB6 -> PB13
- J6 pad 2: PB7 -> PB12
- J6 pad 3: PB8 -> PB11
- J6 pad 4: PB9 -> PB10
- J6 pad 5: PB10 -> PB2
- J7 pad 1: PB11 -> PB5
- J7 pad 2: PB12 -> PB6
- J7 pad 3: PB13 -> PB7
- J7 pad 4: PB14 -> PB8
- J7 pad 5: PB15 -> PB9
- U1 pad 2: unconnected-(U1-PC13-Pad2) -> STATUS_LED
- U1 pad 3: unconnected-(U1-PC14-Pad3) -> USER_BTN
Routing:
- net NRST: track 0.00 -> 55.7 mm, vias 0 -> 2
- net USER_BTN: track 0.00 -> 40.8 mm, vias 0 -> 1
- net +3V3: track 0.00 -> 36.7 mm, vias 0 -> 16
- net GND: track 0.00 -> 31.8 mm, vias 0 -> 90
- net USART1_RX: track 0.00 -> 30.7 mm, vias 0 -> 1
- net USART1_TX: track 0.00 -> 30.4 mm, vias 0 -> 1
- net STATUS_LED: track 0.00 -> 29.9 mm, vias 0 -> 2
- net PB1: track 0.00 -> 29.7 mm
- net PB2: track 0.00 -> 28.9 mm
- net PB5: track 0.00 -> 27.4 mm
- net PB0: track 0.00 -> 26.9 mm
- net PB10: track 0.00 -> 26.1 mm
- net BOOT: track 0.00 -> 24.7 mm, vias 0 -> 2
- net PB6: track 0.00 -> 24.4 mm
- net PB11: track 0.00 -> 24.1 mm
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- added copper zone on B.Cu, net +3V3
- added copper zone on In2.Cu, net +5V
- added copper zone on F.Cu, net GND
- added copper zone on In1.Cu, net GND
- added copper zone on In2.Cu, net GND
Other:
- copper layers 2 -> 4
- board text added: "A0"
- board text added: "A1"
- board text added: "A10"
- board text added: "A11"
- board text added: "A12"
- board text added: "A15"
- board text added: "A4"
- board text added: "A5"
- board text added: "A6"
- board text added: "A7"
- board text added: "A8"
- board text added: "A9"
- board text added: "B0"
- board text added: "B1"
- board text added: "B10"
- board text added: "B11"
- board text added: "B12"
- board text added: "B13"
- board text added: "B14"
- board text added: "B15"
- board text added: "B2"
- board text added: "B3"
- board text added: "B4"
- board text added: "B5"
- board text added: "B6"
- board text added: "B7"
- board text added: "B8"
- board text added: "B9"
- board text added: "JLCJLCJLCJLC"
- board text added: "{"

Commit message: soldered and tested hardware
Other:
- board text added: "CppCon 2024"
- board text added: "clk"
- board text added: "dio"
- board text added: "nrst"
Changed lines of the file:
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@@
+    (effects (font (size 0.75 0.75) (thickness 0.1)) (justify left bottom))
+  )
+  (gr_text "nrst" (at 140.725 78.1) (layer "F.SilkS")
     (effects (font (size 0.75 0.75) (thickness 0.1)) (justify left bottom))
   )
@@
     (effects (font (size 1 1) (thickness 0.15)) (justify left bottom))
   )
-  (gr_text "power" (at 145.529 94.996) (layer "F.SilkS")
+  (gr_text "power" (at 145.875 95.225) (layer "F.SilkS")
     (effects (font (size 1 1) (thickness 0.15)) (justify left bottom))
   )
@@
     (effects (font (size 0.75 0.75) (thickness 0.1)) (justify left bottom))
   )
-  (gr_text "boot" (at 132.372 86.106) (layer "F.SilkS")
+  (gr_text "boot" (at 133.825 86.106) (layer "F.SilkS")
     (effects (font (size 1 1) (thickness 0.15)) (justify left bottom))
   )
@@
     (effects (font (size 0.75 0.75) (thickness 0.1)) (justify left bottom))
   )
-  (gr_text "{" (at 136.4 101.9) (layer "F.SilkS")
-    (effects (font (size 3 3) (thickness 0.45)) (justify left bottom))
+  (gr_text "{" (at 131.1 98.85) (layer "F.SilkS")
+    (effects (font (size 4 4) (thickness 0.6)) (justify left bottom))
   )
   (gr_text "B3" (at 151.403571 98.2375) (layer "F.SilkS")
@@
     (effects (font (size 0.75 0.75) (thickness 0.1)) (justify left bottom))
   )
+  (gr_text "CppCon 2024" (at 129.1 119.9) (layer "F.SilkS")
+    (effects (font (size 2 2) (thickness 0.3)) (justify left bottom))
+  )
   (gr_text "tx" (at 136.182 138.938) (layer "F.SilkS")
     (effects (font (size 1 1) (thickness 0.15)) (justify left bottom))
   )
+  (gr_text "dio" (at 143.675 78.1) (layer "F.SilkS")
+    (effects (font (size 0.75 0.75) (thickness 0.1)) (justify left bottom))
+  )
+  (gr_text "clk" (at 146.075 78.1) (layer "F.SilkS")
+    (effects (font (size 0.75 0.75) (thickness 0.1)) (justify left bottom))
+  )
   (dimension (type aligned) (layer "User.1")
