File: hardware/hardware.kicad_sch (KiCad schematic)
At the start: 53 parts, among them J1 SWD, J2 serial, J3 analog, J4 digital_0, J5 digital_1, J6 digital_2, J7 digital_3, J8 power_0, J9 power_1, SW1 reset_btn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

Commit message: ordering first prototype
Connections:
- net PA10: now also J4.1 (Pin_1); no longer J4.3 (Pin_3)
- net PA11: now also J5.5 (Pin_5); no longer J4.2 (Pin_2)
- net PA12: now also J5.4 (Pin_4); no longer J4.1 (Pin_1)
- net PA15: now also J5.3 (Pin_3); no longer J5.4 (Pin_4)
- net PA8: now also J4.3 (Pin_3); no longer J4.5 (Pin_5)
- net PA9: now also J4.2 (Pin_2); no longer J4.4 (Pin_4)
- net PB10: now also J6.4 (Pin_4); no longer J6.5 (Pin_5)
- net PB11: now also J6.3 (Pin_3); no longer J7.1 (Pin_1)
- net PB12: now also J6.2 (Pin_2); no longer J7.2 (Pin_2)
- net PB13: now also J6.1 (Pin_1); no longer J7.3 (Pin_3)
- net PB14: now also J4.5 (Pin_5); no longer J7.4 (Pin_4)
- net PB15: now also J4.4 (Pin_4); no longer J7.5 (Pin_5)
- net PB2: now also J6.5 (Pin_5); no longer J5.5 (Pin_5)
- net PB3: now also J5.2 (Pin_2); no longer J5.3 (Pin_3)
- net PB4: now also J5.1 (Pin_1); no longer J5.2 (Pin_2)
- net PB5: now also J7.1 (Pin_1); no longer J5.1 (Pin_1)
- net PB6: now also J7.2 (Pin_2); no longer J6.1 (Pin_1)
- net PB7: now also J7.3 (Pin_3); no longer J6.2 (Pin_2)
- net PB8: now also J7.4 (Pin_4); no longer J6.3 (Pin_3)
- net PB9: now also J7.5 (Pin_5); no longer J6.4 (Pin_4)
- net STATUS_LED: now also U1.2 (PC13)
- net USER_BTN: now also U1.3 (PC14)
- no-connect marks 7 -> 5
Other:
- moved on the sheet: C1, C10, C11, C12, C13, C14, C15, C16, C17, C18, C2, C3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

Commit message: soldered and tested hardware
Parts:
- C1, C2: LCSC part number C2857965 -> (none); in the shopping cart y -> (none)
- C10, C14, C15, C16, C17, C7: LCSC Part # C14663 -> (none); TODO OK -> (none); found (none) -> y
- C11, C12: LCSC Part # C182482 -> (none); TODO OK -> (none); found (none) -> y
- C13: LCSC Part # C19666 -> (none); TODO OK -> (none); found (none) -> y
- C18, C3, C5: LCSC part number C880609 -> (none); in the shopping cart y -> (none)
- C4: LCSC part number C2857985 -> (none); in the shopping cart y -> (none)
- C6: LCSC part number C967571 -> (none); in the shopping cart y -> (none)
- C8: LCSC Part # C15849 -> (none); TODO OK -> (none); found (none) -> y
- C9: LCSC Part # C57112 -> (none); TODO OK -> (none); found (none) -> y
- D1: LCSC part number C130722 -> (none); in the shopping cart y -> (none)
- D2: LCSC part number C130724 -> (none); in the shopping cart y -> (none)
- D3: LCSC part number C2892494 -> (none); found y -> (none); in the shopping cart y -> (none)
- D4: LCSC part number C316049 -> (none); found y -> (none); in the shopping cart y -> (none)
- D5: LCSC Part # C72043 -> (none); TODO OK -> (none); found (none) -> y
- L1: LCSC Part # C75654 -> (none); TODO OK -> (none); found (none) -> y
- R1, R4: LCSC part number C3015825 -> (none); in the shopping cart y -> (none)
- R10: LCSC Part # C23182 -> (none); TODO OK -> (none); found (none) -> y
- R2, R3: LCSC part number C3015799 -> (none); in the shopping cart y -> (none)
- R5, R6, R7: LCSC Part # C23345 -> (none); TODO OK -> (none); found (none) -> y
- R8: LCSC Part # C22940 -> (none); TODO OK -> (none); found (none) -> y
- R9: LCSC Part # C25804 -> (none); TODO OK -> (none); found (none) -> y
- SW1, SW2: LCSC part number C221897 -> (none); in the shopping cart y -> (none)
- SW3: TODO OK -> (none); found (none) -> y
- U1: found (none) -> y
- U2: in the shopping cart got it -> (none)
- Y1: LCSC Part # C13738 -> (none); TODO OK -> (none); found (none) -> y
Other:
- company: (none) -> Marcell Juhasz
- title: (none) -> CppCon 2024
- moved on the sheet: C10, C11, C12, C13, C14, C15, C16, C17, C18, C2, C8, C9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
